Commit message: adding camera plugin

File: vision_rpi_bot/urdf/vision_rpi_bot.urdf (robot description, URDF)
Before this commit: robot Vision_Rpi_Bot, 8 links, 7 joints
Joints:
- joint base_joint: origin xyz=0 0 0.14 rpy=0 0 0 -> xyz=0 0 0.15 rpy=0 0 0
- joint camera_joint: origin xyz=0 0 0.14 rpy=0 0 0 -> xyz=0 -0.18 0.2 rpy=0 0 0
- joint caster_holder_joint: origin xyz=0 0 0.14 rpy=0 0 0 -> xyz=0 -0.19 -0.02 rpy=0 0 0
- joint caster_wheel_joint: origin xyz=0 0 0.14 rpy=0 0 0 -> xyz=0 -0.0029 -0.086 rpy=0 0 0; parent base_link -> caster_holder_link
- joint cover_joint: origin xyz=0 0 0.14 rpy=0 0 0 -> xyz=0 0 0.08 rpy=0 0 0
- joint left_wheel_joint: origin xyz=0 0 0.14 rpy=0 0 0 -> xyz=0.235 0.15 -0.05 rpy=0 0 -1.57
- joint right_wheel_joint: axis 0.0 1 0.0 -> 0.0 -1 0.0; origin xyz=0 0 0.14 rpy=0 0 0 -> xyz=-0.235 0.15 -0.05 rpy=0 0 1.57

Commit message: added lidar gazebo plugin

File: vision_rpi_bot/urdf/vision_rpi_bot.urdf (robot description, URDF)
Before this commit: robot Vision_Rpi_Bot, 8 links, 7 joints
Links:
- link camera_link: mass 10 -> 0.75
Joints:
- joint camera_joint: origin xyz=0 -0.18 0.2 rpy=0 0 0 -> xyz=0 -0.18 0.2 rpy=0.0 0 -1.57

Commit message: added qr_test script

File: vision_rpi_bot/urdf/vision_rpi_bot.urdf (robot description, URDF)
Before this commit: robot Vision_Rpi_Bot, 8 links, 7 joints
Links:
- added link lidar_link
Joints:
- added joint lidar_joint: type fixed, parent base_link, child lidar_link, origin xyz=0 -0.25 0.1 rpy=0.0 0 -3.14
