Commit message: line following update - camera tested

File: vision_rpi_bot/urdf/vision_rpi_bot_lf.urdf (robot description, URDF)
Before this commit: robot Vision_Rpi_Bot, 8 links, 7 joints
Links:
- link base_link: mass 10 -> 4
- link caster_wheel_link: mass 10 -> 1
- link left_wheel_link: mass 10 -> 2
- link right_wheel_link: mass 10 -> 2
